File: KiCad/testboard/testboard/testboard.kicad_sch (KiCad schematic)
At the start: 0 parts

Commit message: テスト用キーボード（途中）
Parts:
- added C1, C2, C3, C4, C5, C6, C7, C8, C9: 0.1uF, Capacitor_SMD:C_0603_1608Metric_Pad1.08x0.95mm_HandSolder, symbol Device:C
- added D1, D10, D12, D14, D16, D18, D4, D6, D8: 1N4148, Diode_THT:D_DO-35_SOD27_P7.62mm_Horizontal, symbol Diode:1N4148
- added D11, D13, D15, D17, D2, D3, D5, D7, D9: SK6812, LED_SMD:LED_SK6812_PLCC4_5.0x5.0mm_P3.2mm, symbol LED:SK6812
- added SW1, SW2, SW3, SW4, SW5, SW6, SW7, SW8, SW9: SW_Push, isw-kbd:CherryMX_Hotswap_1u, symbol Switch:SW_Push
- added U1: RP2040-Zero, RP2040-ZeroSocket:RP2040-ZeroSocket, symbol isw-mcu:RP2040-Zero
Connections:
- new net: D1.1 (K), D4.1 (K), D6.1 (K), U1.26
- new net: D4.2 (A), SW2.2
- new net: D11.4 (DOUT), D13.2 (DIN)
- new net: D13.4 (DOUT), D15.2 (DIN)
- new net: D15.4 (DOUT), D17.2 (DIN)
- new net: SW3.1, SW6.1, SW9.1, U1.0
- new net: D12.2 (A), SW6.2
- new net: D11.2 (DIN), D9.4 (DOUT)
- new net: D6.2 (A), SW3.2
- new net: D18.2 (A), SW9.2
- new net: SW2.1, SW5.1, SW8.1, U1.1
- new net: D10.1 (K), D12.1 (K), D8.1 (K), U1.15
- new net: SW1.1, SW4.1, SW7.1, U1.2
- new net: D1.2 (A), SW1.2
- new net: D7.4 (DOUT), D9.2 (DIN)
- new net: D14.1 (K), D16.1 (K), D18.1 (K), U1.14
- new net: D2.4 (DOUT), D3.2 (DIN)
- new net: D3.4 (DOUT), D5.2 (DIN)
- new net: D5.4 (DOUT), D7.2 (DIN)
- new net: D8.2 (A), SW4.2
- new net: D14.2 (A), SW7.2
- new net: D10.2 (A), SW5.2
- new net: D2.2 (DIN), U1.13
- new net: D16.2 (A), SW8.2
- new net +5V: C1.1, C2.1, C3.1, C4.1, C5.1, C6.1, C7.1, C8.1, C9.1, D11.3 (VDD), D13.3 (VDD), D15.3 (VDD), D17.3 (VDD), D2.3 (VDD), D3.3 (VDD), D5.3 (VDD), D7.3 (VDD), D9.3 (VDD), U1.32 (5V)
- new net GND: C1.2, C2.2, C3.2, C4.2, C5.2, C6.2, C7.2, C8.2, C9.2, D11.1 (VSS), D13.1 (VSS), D15.1 (VSS), D17.1 (VSS), D2.1 (VSS), D3.1 (VSS), D5.1 (VSS), D7.1 (VSS), D9.1 (VSS), U1.31 (GND)
- no-connect marks 0 -> 1
