File: KiCad/testboard/testboard/testboard.kicad_pcb (KiCad board)
At the start: 2 copper layers, 99.5 x 99.7 mm, 31 parts

Commit message: テスト用キーボード（途中）
Parts:
- removed REF** (x30): KEY_SWITCH, isw-kbd:CherryMX_Hotswap_1u
- removed REF**: RP2040-ZeroSocket, RP2040-ZeroSocket:RP2040-ZeroSocket
- added C1: 0.1uF, Capacitor_SMD:C_0603_1608Metric_Pad1.08x0.95mm_HandSolder, F.Cu at (93.9, 22.9)
- added C2: 0.1uF, Capacitor_SMD:C_0603_1608Metric_Pad1.08x0.95mm_HandSolder, F.Cu at (93.9, 25.4)
- added C3: 0.1uF, Capacitor_SMD:C_0603_1608Metric_Pad1.08x0.95mm_HandSolder, F.Cu at (93.9, 27.9)
- added C4: 0.1uF, Capacitor_SMD:C_0603_1608Metric_Pad1.08x0.95mm_HandSolder, F.Cu at (93.9, 30.4)
- added C5: 0.1uF, Capacitor_SMD:C_0603_1608Metric_Pad1.08x0.95mm_HandSolder, F.Cu at (93.9, 32.9)
- added C6: 0.1uF, Capacitor_SMD:C_0603_1608Metric_Pad1.08x0.95mm_HandSolder, F.Cu at (93.9, 35.4)
- added C7: 0.1uF, Capacitor_SMD:C_0603_1608Metric_Pad1.08x0.95mm_HandSolder, F.Cu at (93.9, 37.9)
- added C8: 0.1uF, Capacitor_SMD:C_0603_1608Metric_Pad1.08x0.95mm_HandSolder, F.Cu at (93.9, 40.4)
- added C9: 0.1uF, Capacitor_SMD:C_0603_1608Metric_Pad1.08x0.95mm_HandSolder, F.Cu at (93.9, 42.9)
- added D1: 1N4148, Diode_THT:D_DO-35_SOD27_P7.62mm_Horizontal, F.Cu at (82.5, 23.4)
- added D10: 1N4148, Diode_THT:D_DO-35_SOD27_P7.62mm_Horizontal, F.Cu at (82.5, 37.6)
- added D11: SK6812, LED_SMD:LED_SK6812_PLCC4_5.0x5.0mm_P3.2mm, F.Cu at (32.5, 98.8)
- added D12: 1N4148, Diode_THT:D_DO-35_SOD27_P7.62mm_Horizontal, F.Cu at (82.5, 41.1)
- added D13: SK6812, LED_SMD:LED_SK6812_PLCC4_5.0x5.0mm_P3.2mm, F.Cu at (40.7, 85.5)
- added D14: 1N4148, Diode_THT:D_DO-35_SOD27_P7.62mm_Horizontal, F.Cu at (82.5, 44.7)
- added D15: SK6812, LED_SMD:LED_SK6812_PLCC4_5.0x5.0mm_P3.2mm, F.Cu at (40.7, 92.1)
- added D16: 1N4148, Diode_THT:D_DO-35_SOD27_P7.62mm_Horizontal, F.Cu at (82.5, 48.2)
- added D17: SK6812, LED_SMD:LED_SK6812_PLCC4_5.0x5.0mm_P3.2mm, F.Cu at (40.7, 98.8)
- added D18: 1N4148, Diode_THT:D_DO-35_SOD27_P7.62mm_Horizontal, F.Cu at (82.5, 51.8)
- added D2: SK6812, LED_SMD:LED_SK6812_PLCC4_5.0x5.0mm_P3.2mm, F.Cu at (24.4, 85.5)
- added D3: SK6812, LED_SMD:LED_SK6812_PLCC4_5.0x5.0mm_P3.2mm, F.Cu at (24.4, 92.1)
- added D4: 1N4148, Diode_THT:D_DO-35_SOD27_P7.62mm_Horizontal, F.Cu at (82.5, 26.9)
- added D5: SK6812, LED_SMD:LED_SK6812_PLCC4_5.0x5.0mm_P3.2mm, F.Cu at (24.4, 98.8)
- added D6: 1N4148, Diode_THT:D_DO-35_SOD27_P7.62mm_Horizontal, F.Cu at (82.5, 30.5)
- added D7: SK6812, LED_SMD:LED_SK6812_PLCC4_5.0x5.0mm_P3.2mm, F.Cu at (32.5, 85.5)
- added D8: 1N4148, Diode_THT:D_DO-35_SOD27_P7.62mm_Horizontal, F.Cu at (82.5, 34.0)
- added D9: SK6812, LED_SMD:LED_SK6812_PLCC4_5.0x5.0mm_P3.2mm, F.Cu at (32.5, 92.1)
- added SW1: SW_Push, isw-kbd:CherryMX_Hotswap_1u, F.Cu at (136.5, 39.0)
- added SW2: SW_Push, isw-kbd:CherryMX_Hotswap_1u, F.Cu at (156.0, 39.0)
- added SW3: SW_Push, isw-kbd:CherryMX_Hotswap_1u, F.Cu at (175.5, 39.0)
- added SW4: SW_Push, isw-kbd:CherryMX_Hotswap_1u, F.Cu at (136.5, 58.5)
- added SW5: SW_Push, isw-kbd:CherryMX_Hotswap_1u, F.Cu at (156.0, 58.5)
- added SW6: SW_Push, isw-kbd:CherryMX_Hotswap_1u, F.Cu at (175.5, 58.5)
- added SW7: SW_Push, isw-kbd:CherryMX_Hotswap_1u, F.Cu at (136.5, 78.0)
- added SW8: SW_Push, isw-kbd:CherryMX_Hotswap_1u, F.Cu at (156.0, 78.0)
- added SW9: SW_Push, isw-kbd:CherryMX_Hotswap_1u, F.Cu at (175.5, 78.0)
- added U1: RP2040-Zero, RP2040-ZeroSocket:RP2040-ZeroSocket, F.Cu at (91.5, 65.9)
Other:
- board size 99.5 x 99.7 mm -> 99.1 x 99.1 mm

Commit message: 3号機発注
Parts:
- moved D2 120.6 mm to (137.2, 42.9)
Changed lines of the file:
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@@
 	(footprint "LED_SMD:LED_SK6812_PLCC4_5.0x5.0mm_P3.2mm"
 		(layer "F.Cu")
-		(at 24.415 85.515)
+		(at 137.25 42.85)
 		(descr "5.0mm x 5.0mm Addressable RGB LED NeoPixel, https://cdn-shop.adafruit.com/product-files/1138/SK6812+LED+datasheet+.pdf")
 		(tags "LED RGB NeoPixel PLCC-4 5050")
